File: rrCrossing_pnp.kicad_sch (KiCad schematic)
At the start: 11 parts, among them Q1 Q_PNP, Q2 Q_PNP

Commit message: Added useful notes
Other:
- note added: ".tran 0.1ms 5s uic .ic V(/Q1_B)=4.3 .ic V(/Q2_B)=5"
- note added: "Generic transistor model did not work. The detail of a better model is required."
- note added: "Learn the node name syntax from the spice netlist Forward Slash is used with a label."
- note added: "Watch out for pin numbers not matching the netlist. See Pin Assignments tab in the components properties Simulation Model."
- note removed: ".tran 0.1ms 5s uic .ic V(/Q1_B)=4.2 .ic V(/Q2_B)=5"
Changed lines of the file:
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@@
 	(generator_version "9.0")
 	(paper "A4")
-	(text ".tran 0.1ms 5s uic\n.ic V(/Q1_B)=4.2\n.ic V(/Q2_B)=5\n\n"
+	(text "Watch out for pin numbers not matching the netlist.\nSee Pin Assignments tab in the components properties Simulation Model."
+		(exclude_from_sim no)
+		(at 195.072 98.806 0)
+		(effects
+			(font
+				(size 0.889 0.889)
+			)
+			(justify left)
+		)
+	)
+	(text "Generic transistor model did not work.\nThe detail of a better model is required."
+		(exclude_from_sim no)
+		(at 186.182 75.946 0)
+		(effects
+			(font
+				(size 0.889 0.889)
+			)
+			(justify left)
+		)
+	)
+	(text "Learn the node name syntax from the spice netlist\nForward Slash is used with a label."
+		(exclude_from_sim no)
+		(at 147.32 54.864 0)
+		(effects
+			(font
+				(size 0.889 0.889)
+			)
+			(justify left)
+		)
+	)
+	(text ".tran 0.1ms 5s uic\n.ic V(/Q1_B)=4.3\n.ic V(/Q2_B)=5\n\n"
 		(exclude_from_sim no)
 		(at 127 57.404 0)
